File: KiCad/projects/Acelerografo_ESP32/Acelerografo_ESP32.kicad_pcb (KiCad board)
At the start: 2 copper layers, 101.5 x 90 mm, 63 parts, among them J1 Conn_01x02, J17 Conn_01x05_Pin, J18 Conn_01x05_Pin, J6 Conn_01x04_Pin, J7 USB_C_Receptacle, SW1 SW_Push, SW2 SW_Push, U1 ESP32-WROOM-32, U2 DS3231M, U3 ADXL355Z, U4 LD1117S33TR_SOT223, U5 MP2307, U6 CH340G, U7 74LVC125

Commit message: Cambio Fuente de Alimentacion Modulo MP2307 y archivo JLPCB
Parts:
- removed C1, C4: 100nF, Capacitor_SMD:C_0402_1005Metric
- removed C2: 10uF, Capacitor_SMD:CP_Elec_4x5.4
- removed C3, C7: 12uF, Capacitor_SMD:CP_Elec_10x12.5
- removed C5: 4.7nF, Capacitor_SMD:C_0402_1005Metric
- removed C6: 10nF, Capacitor_SMD:C_0402_1005Metric
- removed L1: 2uH, LibsRSA:IND-SMD_L6.0-W6.0_FNR60XXS
- removed R1, R3: 8.2k, Resistor_SMD:R_0805_2012Metric
- removed R2: 100k, Resistor_SMD:R_1206_3216Metric
- removed RVe1: 200k, LibsRSA:RES-ADJ-SMD_3P-L3.4-W3.1_JER33X-1-24
- removed U5: MP2307, Package_SO:SOIC-8_3.9x4.9mm_P1.27mm
- added C20: 220uF, Capacitor_SMD:CP_Elec_4x5.4, F.Cu at (165.0, 40.0)
- added C21: 100nF, Capacitor_SMD:C_0402_1005Metric, F.Cu at (172.5, 40.0)
- added C22: 100uF, Capacitor_SMD:CP_Elec_4x5.4, F.Cu at (186.2, 37.3)
- added C23: 100nF, Capacitor_SMD:C_0402_1005Metric, F.Cu at (185.9, 44.7)
- added C24: 10nF, Capacitor_SMD:C_0402_1005Metric, F.Cu at (185.9, 48.3)
- added J13: Conn_01x01_Pin, Connector_PinHeader_2.54mm:PinHeader_1x01_P2.54mm_Vertical, F.Cu at (185.9, 63.5)
- added J16: Conn_01x01_Pin, Connector_PinHeader_2.54mm:PinHeader_1x01_P2.54mm_Vertical, F.Cu at (177.5, 95.6)
- added J9: IN_LD, Connector_PinHeader_2.54mm:PinHeader_1x01_P2.54mm_Vertical, F.Cu at (203.2, 46.7)
- added U8: STEP_DOWN_CONVERTER, LibsExt:STEP_DOWN_CONVERTER, F.Cu at (163.8, 58.0)
- moved R12 17.6 mm to (195.1, 89.7)
- moved C18 9.02 mm to (185.2, 100.1)
- moved C19 9.02 mm to (187.7, 100.1)
- moved D7 9.02 mm to (211.6, 105.1)
- moved R10 9.02 mm to (192.2, 85.4)
- moved R11 9.02 mm to (185.7, 105.6)
- moved R14 9.02 mm to (191.2, 101.6)
- moved R15 9.02 mm to (191.2, 97.6)
- moved R16 9.02 mm to (209.7, 98.1)
- moved R17 9.02 mm to (209.7, 101.6)
- moved R18 9.02 mm to (217.7, 106.6)
- moved U2 9.02 mm to (200.2, 102.6)
- moved U7 9.02 mm to (185.7, 89.9)
- moved D4 8.98 mm to (175.6, 77.5)
- moved R8 8.63 mm to (170.0, 77.5)
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- renumbered J1 to 12V1, SW1 to EN1, SW2 to RTS1
Connections:
- 12V1 pad 2: /IN_MP2307 -> Net-(12V1-Pin_2)
Routing:
- net Net-(12V1-Pin_2): track 0.00 -> 253.0 mm
- net /IN_MP2307: track 122.1 -> 0.00 mm, vias 3 -> 0
- net GND: track 530.7 -> 615.2 mm, vias 1 -> 0
- net VCC: track 283.0 -> 344.2 mm, vias 5 -> 4
- net Net-(D1-K): track 42.2 -> 73.5 mm
- net Net-(U5-FB): track 26.3 -> 0.00 mm
- net /RXD0-ESP: track 94.8 -> 68.5 mm, vias 2 -> 1
- net /D+: track 35.3 -> 11.9 mm, vias 2 -> 0
- net Net-(D1-A): track 46.7 -> 65.4 mm
- net Net-(U5-SW): track 17.7 -> 0.00 mm
- net Net-(U5-SS): track 17.3 -> 0.00 mm
- net /SCK: track 53.8 -> 40.5 mm
- net /EN_MP2307: track 12.0 -> 0.00 mm
- net Net-(R11-Pad2): track 13.2 -> 24.5 mm
- net /MOSI: track 60.1 -> 50.4 mm
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- added copper zone on B.Cu, net GND
- added copper zone on F.Cu, net GND
