File: KiCad/projects/Acelerografo_ESP32/Acelerografo_ESP32.kicad_sch (KiCad schematic)
At the start: 76 parts, among them J1 Conn_01x02, J10 Conn_01x02_Pin, J11 Conn_01x01_Pin, J12 Conn_01x02_Pin, J13 Conn_01x01_Pin, J14 Conn_01x01_Pin, J15 Conn_01x01_Pin, J16 Conn_01x01_Pin, J17 Conn_01x05_Pin, J18 Conn_01x05_Pin, J2 Conn_01x01_Pin, J3 Conn_01x01_Pin, J4 Conn_01x01_Pin, J5 Conn_01x01_Pin, J6 Conn_01x04_Pin, J7 USB_C_Receptacle, J8 Conn_01x01_Pin, J9 Conn_01x01_Pin, U1 ESP32-WROOM-32, U2 DS3231M, U3 ADXL355Z, U4 LD1117S33TR_SOT223, U5 MP2307, U6 CH340G, U7 74LVC125

Commit message: Cambio Fuente de Alimentacion Modulo MP2307 y archivo JLPCB
Parts:
- removed C1, C4: 100nF, Capacitor_SMD:C_0402_1005Metric, symbol Device:C
- removed C2: 10uF, Capacitor_SMD:CP_Elec_4x5.4, symbol Device:C_Polarized
- removed C3, C7: 12uF, Capacitor_SMD:CP_Elec_10x12.5, symbol Device:C_Polarized
- removed C5: 4.7nF, Capacitor_SMD:C_0402_1005Metric, symbol Device:C
- removed C6: 10nF, Capacitor_SMD:C_0402_1005Metric, symbol Device:C
- removed J10, J12: Conn_01x02_Pin, Connector_PinHeader_2.54mm:PinHeader_1x02_P2.54mm_Vertical, symbol Connector:Conn_01x02_Pin
- removed J11, J14, J15, J2, J3, J4, J5, J8: Conn_01x01_Pin, Connector_PinHeader_2.54mm:PinHeader_1x01_P2.54mm_Vertical, symbol Connector:Conn_01x01_Pin
- removed L1: 2uH, LibsRSA:IND-SMD_L6.0-W6.0_FNR60XXS, symbol Device:L
- removed R1, R3: 8.2k, Resistor_SMD:R_0805_2012Metric, symbol Device:R
- removed R2: 100k, Resistor_SMD:R_1206_3216Metric, symbol Device:R
- removed RVe1: 200k, LibsRSA:RES-ADJ-SMD_3P-L3.4-W3.1_JER33X-1-24, symbol Device:R_Potentiometer_Trim
- removed U5: MP2307, Package_SO:SOIC-8_3.9x4.9mm_P1.27mm, symbol LibsExt:MP2307
- added C20: 220uF, Capacitor_SMD:CP_Elec_4x5.4, symbol Device:C_Polarized
- added C21, C23: 100nF, Capacitor_SMD:C_0402_1005Metric, symbol Device:C
- added C22: 100uF, Capacitor_SMD:CP_Elec_4x5.4, symbol Device:C_Polarized
- added C24: 10nF, Capacitor_SMD:C_0402_1005Metric, symbol Device:C
- added U8: STEP_DOWN_CONVERTER, LibsExt:STEP_DOWN_CONVERTER, symbol LibsExt:root_0_STEP_DOWN_CONVERTER_Micelaneos.SchLib
- J9: value Conn_01x01_Pin -> IN_LD
- renumbered J1 to 12V1, EN to EN1, RTS to RTS1
Connections:
- net GND: now also C20.2, C21.2, C22.2, C23.2, C24.2, U8.2 (IN-), U8.4 (OUT-); no longer J9.1 (Pin_1)
- net at C10.1, C8.1, C9.1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: now also J9.1 (Pin_1)
- net at D1.2 (A), R4.1: now also C22.1, C23.1, C24.1, U8.3 (OUT+)
- net IN_MP2307: no longer names the net of 12V1.2 (Pin_2)
- net IN_MP2307: now also C20.1, C21.1, U8.1 (IN+)
Other:
- moved on the sheet: 12V1, D1
